Commit message: thinh

File: ur10e_with_rg2/ur10e_robot.urdf (robot description, URDF)
Before this commit: robot ur10e_rg2, 18 links, 17 joints
Links:
- removed link left_inner_finger
- removed link left_inner_knuckle
- removed link left_outer_knuckle
- removed link onrobot_rg2_base_link
- removed link right_inner_finger
- removed link right_inner_knuckle
- removed link right_outer_knuckle
- added link world
Joints:
- removed joint finger_joint
- removed joint left_inner_finger_joint
- removed joint left_inner_knuckle_joint
- removed joint right_inner_finger_joint
- removed joint right_inner_knuckle_joint
- removed joint right_outer_knuckle_joint
- removed joint tool0-rg2
- added joint world_joint: type fixed, parent world, child base_link, origin xyz=0.0 0.0 0.77 rpy=0.0 0.0 0.0
- joint base_link-base_fixed_joint: origin rpy=0 0 -3.141593 -> xyz=0 0 0 rpy=0 0 -3.14159265359
